File: PCB/HanaLinear.kicad_pcb (KiCad board)
At the start: 2 copper layers, 179 parts, among them J1 USB_C_Receptacle_USB2.0_14P, J2 SW, SW1 Esc, SW10 3, SW11 4, SW12 5, SW13 6, SW14 7, SW15 8, SW16 9, SW17 0, SW18 -, SW19 =, SW2 F3, SW20 Delete, SW21 Brightness, SW22 Volume, SW23 Tab, SW24 Q, SW25 W, SW26 E, SW27 R, SW28 T, SW29 Y, SW3 F4, SW30 U, SW31 I, SW32 O, SW33 P, SW34 [, SW35 ], SW36 |, SW37 CapsLock, SW38 A, SW39 S, SW4 F7, SW40 D, SW41 F, SW42 G, SW43 H, SW44 J, SW45 K, SW46 L, SW47 ;, SW48 ', SW49 Return, SW5 F8, SW50 Left Shift, SW51 Z, SW52 X, SW53 C, SW54 V, SW55 B, SW56 N, SW57 M, SW58 ,, SW59 ., SW6 F9, SW60 /, SW61 Right Shift, SW62 Fn, SW63 Control, SW64 Option, SW65 Command, SW66 Space, SW67 Left, SW68 Down, SW69 Up, SW7 `, SW70 Right, SW71 BOOTSEL, SW72 RESET, SW73 USB_BOOT, SW8 1, SW9 2, U1 NCP1117-3.3_SOT223, U2 W25Q128JVS, U3 RP2040, Y1 ABM8-272-T3

Commit message: :3c
Parts:
- D1, D10, D11, D12, D13, D14, D15, D16, D17, D18, D19, D2, D20, D21, D22, D23, D24, D25, D26, D27, D28, D29, D3, D30, D31, D32, D33, D34, D35, D36, D37, D38, D39, D4, D40, D41, D42, D43, D44, D45, D46, D47, D48, D49, D5, D50, D51, D52, D53, D54, D55, D56, D57, D58, D59, D6, D60, D61, D62, D63, D64, D65, D66, D67, D68, D7, D8, D9: moved to B.Cu
- moved D68 457.6 mm to (543.8, 342.1), turned to 90 degrees
- moved D34 451.6 mm to (543.8, 284.9), turned to 90 degrees
- moved D59 443.5 mm to (534.2, 323.0), turned to 90 degrees
- moved D47 442.4 mm to (534.2, 303.9), turned to 90 degrees
- moved D67 441.9 mm to (524.7, 342.1), turned to 90 degrees
- moved SW21 440.2 mm to (535.8, 188.2), turned to 180 degrees
- moved D20 439.3 mm to (534.2, 265.9), turned to 90 degrees
- moved D33 434.8 mm to (524.7, 284.9), turned to 90 degrees
- moved D66 426.6 mm to (505.7, 342.1), turned to 90 degrees
- moved SW22 419.1 mm to (485.6, 251.0), turned to 180 degrees
- moved D58 418.9 mm to (505.7, 323.0), turned to 90 degrees
- moved D32 418.3 mm to (505.7, 284.9), turned to 90 degrees
- moved D46 417.2 mm to (505.7, 303.9), turned to 90 degrees
- moved D19 412.7 mm to (505.7, 265.9), turned to 90 degrees
- moved D65 411.6 mm to (486.6, 342.1), turned to 90 degrees
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Routing:
- net ROW6: track 0.00 -> 266.7 mm
- net ROW2: track 0.00 -> 257.2 mm
- net ROW3: track 0.00 -> 257.2 mm
- net ROW4: track 0.00 -> 247.7 mm
- net ROW5: track 0.00 -> 238.1 mm
- net ROW1: track 0.00 -> 161.9 mm
- net Net-(D48-A): track 0.00 -> 63.3 mm
- net Net-(D33-K): track 0.00 -> 55.1 mm
- net Net-(D35-K): track 0.00 -> 43.2 mm
- net Net-(D36-K): track 0.00 -> 40.3 mm
- net Net-(D21-A): track 0.00 -> 25.1 mm
- net Net-(D20-K): track 0.00 -> 25.1 mm
- net Net-(D59-K): track 0.00 -> 25.1 mm
- net Net-(D34-K): track 0.00 -> 25.1 mm
- net Net-(D1-K): track 0.00 -> 23.4 mm
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- added copper zone on B.Cu, net GND
- added copper zone on F.Cu, net GND
Other:
- board outline added: 300 x 138.9 mm

Commit message: glnsalfjnds,f
Parts:
- removed C18: 0.001uF, Capacitor_SMD:C_0201_0603Metric
- removed R8: 1M, Resistor_SMD:R_0201_0603Metric
- C11, C13, C14, C17, C20, C9, R1, R3, R4, R6, R9, U2, U3, Y1: moved to B.Cu
- SW: renamed from J2; moved to B.Cu
- moved H3 480.8 mm to (566.3, 353.9)
- moved H2 437.2 mm to (566.3, 218.0)
- moved U1 305.6 mm to (413.6, 226.3), turned to 180 degrees
- moved C16 297.2 mm to (418.6, 227.5), turned to -90 degrees
- moved SW71 254.2 mm to (297.8, 229.2)
- moved H4 250.9 mm to (271.3, 353.9)
- moved SW72 241.2 mm to (287.7, 229.1)
- moved SW73 224.5 mm to (271.4, 229.3), turned to 180 degrees
- moved C17 218.1 mm to (274.4, 241.9), turned to 180 degrees
- moved C4 213.6 mm to (281.3, 231.2), turned to 90 degrees
- moved C1 213.5 mm to (276.8, 230.0), turned to -90 degrees
- moved C5 213.1 mm to (279.8, 233.6), turned to -90 degrees
- moved C3 212.6 mm to (280.4, 228.9)
- moved R2 212.1 mm to (281.7, 235.1), turned to -90 degrees
- moved C20 211.6 mm to (271.7, 239.3), turned to -90 degrees
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Connections:
- net Net-(U3-VREG_VOUT) renamed +1V1
- C1 pad 1: Net-(U3-ADC_AVDD) -> +3V3
- C10 pad 2: Net-(U3-ADC_AVDD) -> +3V3
- C12 pad 2: Net-(U3-ADC_AVDD) -> +3V3
- C2 pad 1: Net-(U3-ADC_AVDD) -> +3V3
- C3 pad 2: Net-(U3-ADC_AVDD) -> +3V3
- C4 pad 1: Net-(U3-ADC_AVDD) -> +3V3
- C5 pad 2: Net-(U3-ADC_AVDD) -> +3V3
- C6 pad 1: Net-(U3-ADC_AVDD) -> +3V3
- C7 pad 2: Net-(U3-ADC_AVDD) -> +3V3
- C8 pad 1: Net-(U3-ADC_AVDD) -> +3V3
- J1 pad S1: Net-(J1-SHIELD) -> GND
- SW21 pad SH: (no net) -> GND
- SW22 pad SH: (no net) -> GND
- U3 pad 1: Net-(U3-ADC_AVDD) -> +3V3
- U3 pad 10: Net-(U3-ADC_AVDD) -> +3V3
- U3 pad 22: Net-(U3-ADC_AVDD) -> +3V3
- U3 pad 33: Net-(U3-ADC_AVDD) -> +3V3
- U3 pad 42: Net-(U3-ADC_AVDD) -> +3V3
- U3 pad 43: Net-(U3-ADC_AVDD) -> +3V3
- U3 pad 44: Net-(U3-ADC_AVDD) -> +3V3
- U3 pad 48: Net-(U3-ADC_AVDD) -> +3V3
- U3 pad 49: Net-(U3-ADC_AVDD) -> +3V3
Routing:
- net COL15: track 0.00 -> 405.9 mm
- net COL14: track 0.00 -> 384.8 mm
- net COL13: track 0.00 -> 364.8 mm
- net COL12: track 0.00 -> 345.3 mm
- net COL11: track 0.00 -> 333.2 mm
- net COL10: track 0.00 -> 315.5 mm
- net COL9: track 0.00 -> 304.3 mm
- net COL8: track 0.00 -> 266.8 mm
- net COL7: track 0.00 -> 256.9 mm
- net BrightnessB: track 0.00 -> 256.0 mm, vias 0 -> 1
- net VolumeB: track 0.00 -> 251.4 mm, vias 0 -> 1
- net BrightnessA: track 0.00 -> 251.3 mm, vias 0 -> 1
- net VolumeA: track 0.00 -> 243.1 mm, vias 0 -> 1
- net Mute: track 0.00 -> 236.2 mm, vias 0 -> 2
- net COL6: track 0.00 -> 235.7 mm
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Other:
- board size 300 x 138.9 mm -> 315 x 155.9 mm

Commit message: fahh
Parts:
- moved SW71 3.57 mm to (301.3, 229.1)
- moved SW72 3.57 mm to (291.2, 229.1)
- moved R7 2.07 mm to (413.0, 215.1)
- moved C15 2.00 mm to (417.1, 220.1)
- moved C16 2.00 mm to (418.6, 225.5)
- moved J1 2.00 mm to (418.8, 213.7)
- moved R5 2.00 mm to (419.9, 220.3)
- moved U1 2.00 mm to (413.6, 224.3)
- renumbered SW to J2
Routing:
- net Net-(U3-GPIO0): track 18.5 -> 28.6 mm
- net Net-(U3-RUN): track 18.0 -> 27.7 mm
- net Net-(D45-K): track 16.9 -> 21.2 mm
- net Net-(D33-K): track 55.1 -> 59.3 mm
- net GND: track 14.2 -> 10.2 mm, vias 7 -> 8
- net COL10: track 315.5 -> 313.9 mm
- net USB_D+: track 152.7 -> 154.2 mm
- net BrightnessA: track 251.3 -> 249.9 mm
- net COL1: track 126.0 -> 125.0 mm
- net USB_D-: track 151.7 -> 152.7 mm, vias 2 -> 1
- net +3V3: track 190.8 -> 189.9 mm
- net QSPI_SD1: track 28.2 -> 27.5 mm
- net Net-(J1-CC2): track 5.84 -> 6.40 mm

Commit message: sdklafjslkdfj
Routing:
- net BrightnessB: track 256.0 -> 255.4 mm
- net BrightnessA: track 249.9 -> 249.4 mm
- net GND: track 10.2 -> 10.1 mm, vias 8 -> 6

Commit message: gdskfakldf
Parts:
- added REF**: 100nF, Capacitor_SMD:C_0201_0603Metric, F.Cu at (328.9, 223.0)
Routing:
- net +3V3: track 189.9 -> 197.2 mm
Other:
- board text added: "+3v3"
- board text added: "GND"
