File: PCB/HanaLinear.kicad_pcb (KiCad board)
At the start: 2 copper layers, 315 x 155.9 mm, 178 parts, among them J1 USB_C_Receptacle_USB2.0_14P, J2 SW, SW1 Esc, SW10 3, SW11 4, SW12 5, SW13 6, SW14 7, SW15 8, SW16 9, SW17 0, SW18 -, SW19 =, SW2 F3, SW20 Delete, SW21 Brightness, SW22 Volume, SW23 Tab, SW24 Q, SW25 W, SW26 E, SW27 R, SW28 T, SW29 Y, SW3 F4, SW30 U, SW31 I, SW32 O, SW33 P, SW34 [, SW35 ], SW36 |, SW37 CapsLock, SW38 A, SW39 S, SW4 F7, SW40 D, SW41 F, SW42 G, SW43 H, SW44 J, SW45 K, SW46 L, SW47 ;, SW48 ', SW49 Return, SW5 F8, SW50 Left Shift, SW51 Z, SW52 X, SW53 C, SW54 V, SW55 B, SW56 N, SW57 M, SW58 ,, SW59 ., SW6 F9, SW60 /, SW61 Right Shift, SW62 Fn, SW63 Control, SW64 Option, SW65 Command, SW66 Space, SW67 Left, SW68 Down, SW69 Up, SW7 `, SW70 Right, SW71 BOOTSEL, SW72 RESET, SW73 USB_BOOT, SW8 1, SW9 2, U1 NCP1117-3.3_SOT223, U2 W25Q128JVS, U3 RP2040, Y1 ABM8-272-T3

Commit message: adsfjdlfka
Parts:
- C12: moved to B.Cu
- moved R7 11.6 mm to (424.6, 215.6), turned to 90 degrees
- moved REF** 4.38 mm to (325.3, 220.5), turned to -90 degrees
- moved C12 1.10 mm to (274.3, 227.7)
- moved C2 0.80 mm to (274.8, 228.7)
- moved R5 0.33 mm to (419.6, 220.4)
Routing:
- net VBUS: track 14.6 -> 7.31 mm
- net Net-(J1-CC2): track 6.40 -> 0.28 mm
- net GND: track 10.1 -> 4.78 mm
- net ROW2: track 321.9 -> 318.4 mm
- net ROW3: track 346.4 -> 342.9 mm
- net ROW4: track 344.1 -> 340.6 mm
- net ROW5: track 368.0 -> 364.4 mm
- net COL1: track 125.0 -> 121.5 mm
- net ROW6: track 403.2 -> 399.7 mm
- net COL2: track 157.3 -> 153.8 mm
- net VolumeB: track 251.1 -> 254.6 mm
- net +1V1: track 14.1 -> 10.7 mm
- net +3V3: track 197.2 -> 198.9 mm
- net USB_D+: track 154.2 -> 152.6 mm, vias 3 -> 1
- net USB_D-: track 152.7 -> 151.7 mm

Commit message: afdklsjdfkl
Parts:
- removed REF**: 100nF, Capacitor_SMD:C_0201_0603Metric
- J1: footprint Connector_USB:USB_C_Receptacle_Amphenol_12401610E4-2A -> Connector_USB:USB_C_Receptacle_G-Switch_GT-USB-7010ASV
- moved R7 7.81 mm to (417.2, 218.1), turned to -90 degrees
- moved C15 2.52 mm to (415.9, 217.9)
- moved R5 2.29 mm to (420.1, 218.1)
- moved J1 1.21 mm to (418.8, 212.5)
- moved C3 0.73 mm to (280.8, 229.6), turned to 90 degrees
Connections:
- SW21 pad SH: GND -> (no net)
- SW22 pad SH: GND -> (no net)
Routing:
- net VBUS: track 7.31 -> 14.3 mm
- net +3V3: track 198.9 -> 194.5 mm
- net +1V1: track 10.7 -> 14.6 mm
- net USB_D+: track 152.6 -> 150.7 mm
- net Net-(J1-CC2): track 0.28 -> 1.64 mm
- net GND: track 4.78 -> 3.56 mm, vias 6 -> 10
- net Net-(U3-GPIO0): track 28.6 -> 27.4 mm
- net ROW3: track 342.9 -> 342.2 mm
- net ROW1: track 182.1 -> 181.5 mm
- net QSPI_SD1: track 27.1 -> 26.6 mm

Commit message: dskjalfjlkf
Parts:
- removed R1: 10K, Resistor_SMD:R_0201_0603Metric
- removed SW71: BOOTSEL, Button_Switch_THT:SW_PUSH_6mm
- U1: value NCP1117-3.3_SOT223 -> AMS1117-3.3
- moved SW73 30.0 mm to (301.3, 229.0), turned to 0 degrees
- moved R6 2.59 mm to (281.2, 209.4), turned to -90 degrees
- moved C16 1.25 mm to (419.0, 224.3), turned to 0 degrees
Connections:
- U3 pad 2: Net-(U3-GPIO0) -> unconnected-(U3-GPIO0-Pad2)
Routing:
- net Net-(U3-GPIO0): track 27.4 -> 0.00 mm
- net Net-(R6-Pad1): track 22.9 -> 44.2 mm
- net +3V3: track 194.5 -> 192.7 mm
- net COL9: track 303.9 -> 305.2 mm
- net GND: vias 10 -> 8

Commit message: dlfksaljfkj
Parts:
- C11, C12, C13, C14, C17, C20, C9, D1, D10, D11, D12, D13, D14, D15, D16, D17, D18, D19, D2, D20, D21, D22, D23, D24, D25, D26, D27, D28, D29, D3, D30, D31, D32, D33, D34, D35, D36, D37, D38, D39, D4, D40, D41, D42, D43, D44, D45, D46, D47, D48, D49, D5, D50, D51, D52, D53, D54, D55, D56, D57, D58, D59, D6, D60, D61, D62, D63, D64, D65, D66, D67, D68, D7, D8, D9, J2, R3, R4, R6, R9, U2, U3, Y1: moved to F.Cu
- moved SW73 33.4 mm to (271.1, 243.2), turned to 180 degrees
- moved SW72 32.2 mm to (271.3, 254.3), turned to 180 degrees
- moved R6 28.9 mm to (271.1, 236.4), turned to 90 degrees
- moved U2 19.7 mm to (268.5, 228.1)
- moved C14 17.7 mm to (270.7, 233.2), turned to 0 degrees
- moved SW21 12.8 mm to (504.8, 251.0), turned to 180 degrees
- moved C5 10.9 mm to (274.2, 224.3), turned to 0 degrees
- moved C12 10.4 mm to (283.3, 222.5), turned to -90 degrees
- moved C1 10.1 mm to (277.9, 220.0), turned to 90 degrees
- moved C2 9.89 mm to (279.4, 220.0), turned to 90 degrees
- moved C3 9.85 mm to (278.7, 220.0), turned to -90 degrees
- moved C20 9.46 mm to (279.6, 234.1), turned to 0 degrees
- moved C4 9.35 mm to (274.2, 225.0), turned to 180 degrees
- moved C10 9.08 mm to (284.0, 222.5), turned to -90 degrees
- moved C17 8.21 mm to (277.1, 234.2)
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Routing:
- net COL15: track 405.9 -> 0.00 mm
- net COL14: track 384.8 -> 0.00 mm
- net COL13: track 364.8 -> 0.00 mm
- net COL12: track 345.3 -> 0.00 mm
- net COL11: track 333.2 -> 0.00 mm
- net COL10: track 313.9 -> 0.00 mm
- net COL9: track 305.2 -> 0.00 mm
- net COL8: track 266.8 -> 0.00 mm
- net COL7: track 256.9 -> 0.00 mm
- net BrightnessB: track 255.4 -> 0.00 mm, vias 1 -> 0
- net VolumeB: track 254.8 -> 0.00 mm, vias 1 -> 0
- net BrightnessA: track 249.4 -> 0.00 mm, vias 1 -> 0
- net VolumeA: track 243.1 -> 0.00 mm, vias 1 -> 0
- net Mute: track 236.4 -> 0.00 mm, vias 2 -> 0
- net COL6: track 235.7 -> 0.00 mm
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