File: PCB/HanaLinear.kicad_pcb (KiCad board)
At the start: 2 copper layers, 315 x 155.9 mm, 175 parts, among them J1 USB_C_Receptacle_USB2.0_14P, J2 SW, SW1 Esc, SW10 3, SW11 4, SW12 5, SW13 6, SW14 7, SW15 8, SW16 9, SW17 0, SW18 -, SW19 =, SW2 F3, SW20 Delete, SW21 Brightness, SW22 Volume, SW23 Tab, SW24 Q, SW25 W, SW26 E, SW27 R, SW28 T, SW29 Y, SW3 F4, SW30 U, SW31 I, SW32 O, SW33 P, SW34 [, SW35 ], SW36 |, SW37 CapsLock, SW38 A, SW39 S, SW4 F7, SW40 D, SW41 F, SW42 G, SW43 H, SW44 J, SW45 K, SW46 L, SW47 ;, SW48 ', SW49 Return, SW5 F8, SW50 Left Shift, SW51 Z, SW52 X, SW53 C, SW54 V, SW55 B, SW56 N, SW57 M, SW58 ,, SW59 ., SW6 F9, SW60 /, SW61 Right Shift, SW62 Fn, SW63 Control, SW64 Option, SW65 Command, SW66 Space, SW67 Left, SW68 Down, SW69 Up, SW7 `, SW70 Right, SW72 RESET, SW73 USB_BOOT, SW8 1, SW9 2, U1 AMS1117-3.3, U2 W25Q128JVS, U3 RP2040, Y1 ABM8-272-T3

Commit message: pcb adkosjfc
Parts:
- moved Y1 1.61 mm to (279.0, 236.4)
- moved C17 0.99 mm to (278.1, 234.1)
- moved C7 0.22 mm to (284.8, 228.4)
Routing:
- net COL15: track 0.00 -> 408.0 mm
- net COL14: track 0.00 -> 337.9 mm
- net COL13: track 0.00 -> 319.3 mm
- net COL12: track 0.00 -> 301.9 mm
- net COL11: track 0.00 -> 269.2 mm
- net COL9: track 0.00 -> 257.4 mm
- net COL10: track 0.00 -> 250.9 mm
- net BrightnessB: track 0.00 -> 250.3 mm
- net COL8: track 0.00 -> 248.9 mm
- net BrightnessA: track 0.00 -> 245.4 mm
- net VolumeB: track 0.00 -> 231.3 mm
- net VolumeA: track 0.00 -> 225.4 mm
- net COL7: track 0.00 -> 209.5 mm
- net Mute: track 0.00 -> 203.7 mm
- net COL6: track 0.00 -> 201.6 mm
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
Commit message: sdfkajlkf
Parts:
- C1, C10, C11, C12, C13, C14, C17, C2, C20, C3, C4, C5, C6, C7, C8, C9: footprint Capacitor_SMD:C_0201_0603Metric -> Capacitor_SMD:C_0402_1005Metric
- R2, R5, R6, R7, R9: footprint Resistor_SMD:R_0201_0603Metric -> Resistor_SMD:R_0402_1005Metric
- R3, R4: footprint Resistor_SMD:R_0201_0603Metric -> Resistor_SMD:R_0603_1608Metric
- moved C17 4.58 mm to (278.4, 238.7), turned to 0 degrees
- moved C20 2.90 mm to (281.7, 236.1), turned to -90 degrees
- moved R4 2.80 mm to (281.9, 219.9)
- moved R3 2.66 mm to (280.4, 219.9)
- moved C1 2.26 mm to (275.7, 220.1)
- moved C3 2.04 mm to (276.7, 220.1)
- moved C2 1.83 mm to (277.6, 220.1)
- moved C10 1.56 mm to (285.6, 222.3)
- moved C12 1.35 mm to (284.6, 222.3)
- moved C9 1.14 mm to (283.6, 222.3)
- moved C5 1.07 mm to (275.3, 224.2), turned to -90 degrees
- moved C13 0.93 mm to (282.6, 222.3)
- moved C4 0.87 mm to (274.3, 224.2), turned to 90 degrees
- moved C8 0.80 mm to (284.6, 225.3), turned to -90 degrees
- moved J2 0.38 mm to (283.8, 233.7)
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Routing:
- net Net-(D26-K): track 16.9 -> 21.2 mm
- net Net-(D11-K): track 17.0 -> 21.2 mm
- net +3V3: track 230.2 -> 232.9 mm
- net Net-(U3-USB_DM): track 1.26 -> 3.49 mm
- net Net-(U3-USB_DP): track 1.43 -> 3.50 mm
- net QSPI_SCLK: track 28.7 -> 30.7 mm
- net Net-(C20-Pad1): track 2.77 -> 3.98 mm
- net Net-(U3-XIN): track 7.71 -> 8.87 mm
- net QSPI_SD3: track 31.3 -> 32.4 mm
- net +1V1: track 14.6 -> 15.6 mm
- net COL15: track 408.0 -> 408.8 mm
- net COL13: track 319.3 -> 320.1 mm
- net COL12: track 301.9 -> 302.7 mm
- net COL14: track 337.9 -> 338.6 mm
- net QSPI_SS: track 19.8 -> 20.5 mm
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Other:
- board text added: "dude i think you broke it"
- board text added: "very linear ineded"
